File: C64 XUM1541/C64 XUM1541.kicad_pcb (KiCad board)
At the start: 2 copper layers, 64.1 x 39.4 mm, 1 part, among them J5 DIN-7

Commit message: Basic module
Parts:
- removed J5: DIN-7, C64_PWR:C64_PWR
- added A1: Arduino_Pro_Micro, arduino_pro_micro:Arduino_Pro_Micro, F.Cu at (108.0, 86.4)
- added D1: POWER, LEDs:LED_D5.0mm, F.Cu at (101.6, 102.2)
- added J1: C64_IEC, C64_IEC:C64_IEC, F.Cu at (74.3, 86.4)
- added R1: 330, Resistors_THT:R_Axial_DIN0207_L6.3mm_D2.5mm_P10.16mm_Horizontal, F.Cu at (88.9, 82.5)
- added SW1: RESET, Buttons_Switches_THT:SW_Tactile_SPST_Angled_PTS645Vx39-2LFS, F.Cu at (116.8, 102.9)
Routing:
- net SRQ: track 0.00 -> 43.4 mm
- net ATN: track 0.00 -> 42.8 mm
- net VCC: track 0.00 -> 37.7 mm
- net DAT: track 0.00 -> 37.5 mm
- net CLK: track 0.00 -> 35.0 mm
- net Net-(D1-Pad2): track 0.00 -> 24.0 mm
- net RST: track 0.00 -> 22.0 mm
- net Net-(A1-Pad22): track 0.00 -> 8.15 mm
- net Net-(A1-Pad9): track 0.00 -> 2.54 mm
- net Net-(A1-Pad8): track 0.00 -> 2.54 mm
- net Net-(A1-Pad7): track 0.00 -> 2.54 mm
- net Net-(A1-Pad6): track 0.00 -> 2.54 mm
- net Net-(A1-Pad5): track 0.00 -> 2.54 mm
- net Net-(A1-Pad2): track 0.00 -> 2.54 mm
- net Net-(A1-Pad10): track 0.00 -> 2.54 mm
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
Commit message: Added parallel header
Parts:
- added J2: PARALLEL, Pin_Headers:Pin_Header_Straight_2x08_Pitch2.54mm, F.Cu at (65.4, 72.4)
Connections:
- A1 pad 1: Net-(A1-Pad1) -> /D3
- A1 pad 17: (no net) -> /D7
- A1 pad 18: (no net) -> /D6
- A1 pad 19: (no net) -> /D5
- A1 pad 2: Net-(A1-Pad2) -> /D2
- A1 pad 20: (no net) -> /D4
- A1 pad 5: Net-(A1-Pad5) -> /D1
- A1 pad 6: Net-(A1-Pad6) -> /D0
Routing:
- net /D4: track 0.00 -> 67.7 mm, vias 0 -> 2
- net /D5: track 0.00 -> 61.4 mm, vias 0 -> 2
- net /D2: track 0.00 -> 55.8 mm
- net /D3: track 0.00 -> 55.0 mm
- net /D1: track 0.00 -> 50.7 mm
- net /D6: track 0.00 -> 50.3 mm, vias 0 -> 2
- net /D0: track 0.00 -> 50.3 mm
- net /D7: track 0.00 -> 44.0 mm, vias 0 -> 2
- net Net-(A1-Pad6): track 2.54 -> 0.00 mm
- net Net-(A1-Pad5): track 2.54 -> 0.00 mm
- net Net-(A1-Pad2): track 2.54 -> 0.00 mm
- net Net-(A1-Pad1): track 2.54 -> 0.00 mm
- net VCC: track 37.7 -> 39.5 mm
- net ATN: track 42.8 -> 41.9 mm
Other:
- board text added: "Revision B"
- board text removed: "Revision A"
